File: contactlessReader_licensed.kicad_pcb (KiCad board)
At the start: 2 copper layers, 95 x 107.1 mm, 38 parts, among them J1 Conn_01x04_Male, J2 Conn_01x08_Male

Commit message: rev. 2.4
Parts:
- removed CRX1: CRX, TestPoint:TestPoint_Pad_1.0x1.0mm
- removed CRX2: CRX2, TestPoint:TestPoint_Pad_1.0x1.0mm
- removed CTX1: CTX, TestPoint:TestPoint_Pad_1.0x1.0mm
- removed CTX2: CTX2, TestPoint:TestPoint_Pad_1.0x1.0mm
- removed Fuse1: Polyfuse, Fuse:Fuse_1206_3216Metric
- removed PWC1: 0.1pF, Capacitor_SMD:C_True_1206_3216Metric
- added AMS1117-5.0: AMS1117-5.0, Package_TO_SOT_SMD:SOT-223-3_TabPin2, F.Cu at (219.9, 123.2)
- added G***: LOGO, AeonLabs:pcbWay Logo Collab, F.Cu at (169.0, 75.5)
- added G***: LOGO, AeonLabs:pcbWay Logo Collab, B.Cu at (166.4, 62.5)
- added LC5: 22uF, Capacitor_SMD:C_1206_3216Metric_Pad1.33x1.80mm_HandSolder, F.Cu at (224.0, 109.4)
- added LC6: 22uF, Capacitor_SMD:C_1206_3216Metric_Pad1.33x1.80mm_HandSolder, F.Cu at (220.8, 116.1)
- added LC7: 100nF, Capacitor_SMD:C_1206_3216Metric_Pad1.33x1.80mm_HandSolder, F.Cu at (224.0, 106.9)
- added LC8: 100nF, Capacitor_SMD:C_1206_3216Metric_Pad1.33x1.80mm_HandSolder, F.Cu at (220.7, 112.9)
- added PWFUSE1: 1A, Fuse:Fuse_1206_3216Metric, F.Cu at (223.9, 104.2)
- added PWR12V1: PWR12V, TerminalBlock_4Ucon:TerminalBlock_4Ucon_1x02_P3.50mm_Vertical, F.Cu at (225.4, 96.7)
- added RX1: RX1, TestPoint:TestPoint_Pad_Bridge_1.0x1.0mm, B.Cu at (168.9, 74.2)
- added TX1: TX1, TestPoint:TestPoint_Pad_Bridge_1.0x1.0mm, B.Cu at (168.9, 71.9)
- added USBFUSE1: 0.5A, Fuse:Fuse_1206_3216Metric, F.Cu at (224.8, 91.9)
- added USB_SCH1: D_Schottky, Diode_SMD:D_1210_3225Metric_Pad1.42x2.65mm_HandSolder, F.Cu at (217.6, 99.9)
- HX4002B1, HX4002B2: footprint Package_SO:SOT95P280X125-6N -> AeonLabs:HX4002 SOT95 P280X125-6N
- moved G*** 85.9 mm to (150.0, 70.6), turned to 0 degrees
- moved G*** 21.3 mm to (163.4, 56.5)
- moved G*** 8.26 mm to (219.1, 60.0)
- moved USB-M1 6.50 mm to (225.7, 84.9)
- moved PC1 5.04 mm to (175.0, 58.4)
- moved PC2 4.78 mm to (174.9, 63.2)
- moved HX4002B2 3.82 mm to (171.3, 62.7)
- moved HX4002B1 3.80 mm to (171.4, 59.0)
- moved BUZZER1 0.36 mm to (167.5, 43.1)
Routing:
- net Net-(AMS1117-5.0-Pad3): track 0.00 -> 36.2 mm, vias 0 -> 6
- net Net-(AMS1117-5.0-Pad1): track 0.00 -> 28.4 mm
- net /5V0: track 143.4 -> 171.1 mm
- net /GND: track 264.8 -> 238.5 mm, vias 12 -> 11
- net Net-(USBFUSE1-Pad1): track 0.00 -> 10.4 mm
- net /5V0F: track 44.0 -> 34.1 mm, vias 2 -> 3
- net /IO16_U2RX_NexTX: track 119.6 -> 113.0 mm
- net /IO17_U2TX_NexRX: track 121.4 -> 114.9 mm
- net /RST_EN_RTS: track 110.9 -> 105.7 mm
- net /IO0_BOOT_DTR: track 125.3 -> 120.8 mm
- net Net-(PWR12V1-Pad2): track 0.00 -> 4.34 mm
- net /IO01TX: track 39.0 -> 35.8 mm
- net /IO03RX: track 38.5 -> 35.4 mm
- net /IO23_RF_MOSI: track 55.8 -> 52.8 mm
- net /RX_IN: track 73.7 -> 71.4 mm
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Other:
- board text added: "0.5A"
- board text added: "1A"
- board text added: "5-12V 1A"
- board text added: "7{dblquote} LCD Touch Addon"
- board text added: "AMS1117"
- board text added: "Contact AeonLabs for a Commercial License"
- board text added: "Copyright CC 2022"
- board text added: "SCH"
- board text added: "USB-M"
- board text added: "board rev. 2.4"
- board text removed: "7{dblquote} LCD Touch"
- board text removed: "Addon for Nextion LCD Touch 7{dblquote}"
- board text removed: "Copyright 2022"
- board text removed: "RESET"
- board text removed: "board rev. 2.3.2"
