File: contactlessReader_licensed.kicad_sch (KiCad schematic)
At the start: 34 parts, among them J1 Conn_01x04_Male, J2 Conn_01x08_Male

Commit message: rev. 2.4
Parts:
- removed CRX1: CRX, TestPoint:TestPoint_Pad_1.0x1.0mm, symbol Connector:TestPoint
- removed CRX2: CRX2, TestPoint:TestPoint_Pad_1.0x1.0mm, symbol Connector:TestPoint
- removed CTX1: CTX, TestPoint:TestPoint_Pad_1.0x1.0mm, symbol Connector:TestPoint
- removed CTX2: CTX2, TestPoint:TestPoint_Pad_1.0x1.0mm, symbol Connector:TestPoint
- removed PWC1: 0.1pF, Capacitor_SMD:C_True_1206_3216Metric, symbol Device:C
- added AMS1117-5.0: AMS1117-5.0, Package_TO_SOT_SMD:SOT-223-3_TabPin2, symbol Regulator_Linear:AMS1117-5.0
- added LC5, LC6: 22uF, Capacitor_SMD:C_1206_3216Metric_Pad1.33x1.80mm_HandSolder, symbol Device:C
- added LC7, LC8: 100nF, Capacitor_SMD:C_1206_3216Metric_Pad1.33x1.80mm_HandSolder, symbol Device:C
- added PWFUSE1: 1A, Fuse:Fuse_1206_3216Metric, symbol Device:Polyfuse
- added PWR12V1: PWR12V, TerminalBlock_4Ucon:TerminalBlock_4Ucon_1x02_P3.50mm_Vertical, symbol Connector:Screw_Terminal_01x02
- added RX1: RX1, TestPoint:TestPoint_Pad_Bridge_1.0x1.0mm, symbol Connector:TestPoint_2Pole
- added TX1: TX1, TestPoint:TestPoint_Pad_Bridge_1.0x1.0mm, symbol Connector:TestPoint_2Pole
- added USB_SCH1: D_Schottky, Diode_SMD:D_1210_3225Metric_Pad1.42x2.65mm_HandSolder, symbol Device:D_Schottky
- HX4002B1, HX4002B2: footprint Package_SO:SOT95P280X125-6N -> AeonLabs:HX4002 SOT95 P280X125-6N
- USBFUSE1: renamed from Fuse1; value Polyfuse -> 0.5A
Connections:
- net 5V0: now also AMS1117-5.0.2 (VO), LC6.1, LC8.1, USB_SCH1.1 (K); no longer USBFUSE1.1
- net IO01TX: now also RX1.2
- net IO03RX: now also TX1.2
- net RX_IN: now also RX1.1
- net TX_IN: now also TX1.1
- new net: USBFUSE1.1, USB_SCH1.2 (A)
- new net: PWFUSE1.1, PWR12V1.2 (Pin_2)
- new net: AMS1117-5.0.3 (VI), LC5.2, LC7.2, PWFUSE1.2
- new net: AMS1117-5.0.1 (GND), LC5.1, LC6.2, LC7.1, LC8.2, PWR12V1.1 (Pin_1)
Other:
- note added: "5V0 LDO and Filtering"
- moved on the sheet: BUZZER1, ENR1, ESP32-WROOM32, ESPC1, ESPC2, ESP_EN_C1, H1, H3, HX4002B1, HX4002B2, ID3V3, IDGND1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
