File: contactlessReader_g.kicad_pcb (KiCad board)
At the start: 2 copper layers, 95 x 107.1 mm, 45 parts, among them J1 Conn_01x04_Male, J2 Conn_01x08_Male

Commit message: revision update
Parts:
- added CH340K1: CH340K1, Package_SO:SSOP-10_3.9x4.9mm_P1.00mm, F.Cu at (197.8, 43.6)
- added CHC1: 100nF, Capacitor_SMD:C_1206_3216Metric, F.Cu at (200.1, 38.4)
- added CHC2: 100nF, Capacitor_SMD:C_1206_3216Metric, F.Cu at (193.8, 41.9)
- added G***: LOGO, AeonLabs:scissors, F.Cu at (228.5, 58.7)
- added G***: LOGO, AeonLabs:Contactless RFID, F.Cu at (171.0, 71.2)
- added G***: LOGO, AeonLabs:Barcode Scanner WiFi Logo, F.Cu at (221.5, 71.7)
- added J3: Conn_01x04_Male, AeonLabs:BarCode Scanner Wireless Receiver PCB Module, F.Cu at (222.6, 55.1)
- moved G*** 76.3 mm to (217.7, 136.3)
- moved G*** 54.4 mm to (114.6, 75.6)
- moved G*** 54.2 mm to (112.3, 66.4)
- moved G*** 5.22 mm to (209.5, 44.0)
- moved PC3 1.08 mm to (165.6, 63.6), turned to 180 degrees
- moved H3 1.02 mm to (224.9, 39.9)
- moved H1 1.02 mm to (225.0, 141.2)
- moved G*** 1.00 mm to (150.9, 70.9)
- moved ESP32-WROOM32 0.09 mm to (148.8, 49.4)
Connections:
- net /IO12_LED_GREEN renamed /IO12_LED_RED
- net /IO13_LED_RED renamed /IO13_LED_GREEN
- ESP32-WROOM32 pad 23: unconnected-(ESP32-WROOM32-Pad23) -> /IO15_U1_RX
- ESP32-WROOM32 pad 31: unconnected-(ESP32-WROOM32-Pad31) -> /IO19_U1_TX
Routing:
- net /IO19_U1_TX: track 0.00 -> 68.4 mm, vias 0 -> 2
- net /IO15_U1_RX: track 0.00 -> 58.9 mm, vias 0 -> 2
- net Net-(CH340K1-Pad1): track 0.00 -> 32.1 mm
- net Net-(CH340K1-Pad2): track 0.00 -> 29.6 mm
- net /5V0: track 171.1 -> 198.1 mm, vias 1 -> 3
- net /GND: track 238.5 -> 258.7 mm, vias 11 -> 13
- net /RST_EN_RTS: track 105.7 -> 109.7 mm
- net /IO0_BOOT_DTR: track 120.8 -> 124.3 mm
- net /IO18_RF_SCK: track 46.1 -> 42.7 mm
- net /TX_IN: track 72.3 -> 75.4 mm
- net Net-(CH340K1-Pad10): track 0.00 -> 3.01 mm
- net /RX_IN: track 71.4 -> 74.2 mm
- net /3V3: track 64.3 -> 61.7 mm
Other:
- board size 95 x 107.1 mm -> 95 x 108.1 mm
- board text added: "LDAD RFID NFC CONTACTLESS WiFi BLE BARCODE SCANNER RECEIVER"
- board text added: "board rev. 3.1"
- board text removed: "LDAD RFID NFC CONTACTLESS WiFi BLE"
- board text removed: "board rev. 2.4"
